File: Hangulator/Hangulator.sch (KiCad schematic (older format))
At the start: 148 parts, among them SW2 SW_Push, U1 ATmega32U4-AU, Y2 Crystal_GND24_Small

Commit message: Working on it more
Parts:
- removed F2: 500mA, Fuse:Fuse_1206_3216Metric_Pad1.42x1.75mm_HandSolder, symbol Device:Polyfuse_Small
- removed R11, R12: 5.1k, Resistor_SMD:R_0805_2012Metric_Pad1.20x1.40mm_HandSolder, symbol Device:R_Small
- removed USB1: HRO-TYPE-C-31-M-12, Type-C:HRO-TYPE-C-31-M-12-HandSoldering, symbol Type-C:HRO-TYPE-C-31-M-12
Connections:
- net +5V: now also U1.24 (AVCC), U1.44 (AVCC); no longer R9.1, U1.2 (UVCC)
- new net: R9.1, U1.2 (UVCC)
Changed lines of the file:
@@
 $EndComp
-Wire Wire Line
-	8900 7400 9000 7400
 Wire Wire Line
 	7750 7950 7750 7850
@@
 	1    8100 8000
 	0    1    1    0
-$EndComp
-$Comp
-L power:+5V #PWR0104
-U 1 1 605502E2
-P 8900 7300
-F 0 "#PWR0104" H 8900 7150 50  0001 C CNN
-F 1 "+5V" H 8915 7473 50  0000 C CNN
-F 2 "" H 8900 7300 50  0001 C CNN
-F 3 "" H 8900 7300 50  0001 C CNN
-	1    8900 7300
-	1    0    0    -1
 $EndComp
 Connection ~ 8900 7350
@@
 	6050 4900 9750 4900
 Connection ~ 6050 4900
-Connection ~ 8900 7400
-Wire Wire Line
-	20925 8925 20300 8925
-Wire Wire Line
-	20925 9825 20300 9825
-Wire Wire Line
-	19975 9275 20100 9275
-Wire Wire Line
-	20300 8925 20300 9275
-Wire Wire Line
-	20300 9825 20300 9275
-Connection ~ 20300 9275
-$Comp
-L Device:Polyfuse_Small F2
-U 1 1 605942C4
-P 20200 9275
-F 0 "F2" V 19995 9275 50  0000 C CNN
-F 1 "500mA" V 20086 9275 50  0000 C CNN
-F 2 "Fuse:Fuse_1206_3216Metric_Pad1.42x1.75mm_HandSolder" H 20250 9075 50  0001 L CNN
-F 3 "~" H 20200 9275 50  0001 C CNN
-	1    20200 9275
-	0    1    1    0
-$EndComp
-$Comp
-L power:+5V #PWR0119
-U 1 1 605942BE
-P 19975 9275
-F 0 "#PWR0119" H 19975 9125 50  0001 C CNN
-F 1 "+5V" H 19990 9448 50  0000 C CNN
-F 2 "" H 19975 9275 50  0001 C CNN
-F 3 "" H 19975 9275 50  0001 C CNN
-	1    19975 9275
-	1    0    0    -1
-$EndComp
-$Comp
-L power:GND #PWR0118
-U 1 1 605942B8
-P 20525 9625
-F 0 "#PWR0118" H 20525 9375 50  0001 C CNN
-F 1 "GND" H 20530 9452 50  0000 C CNN
-F 2 "" H 20525 9625 50  0001 C CNN
-F 3 "" H 20525 9625 50  0001 C CNN
-	1    20525 9625
-	1    0    0    -1
-$EndComp
-$Comp
-L power:GND #PWR0117
-U 1 1 605942B2
-P 20525 9025
-F 0 "#PWR0117" H 20525 8775 50  0001 C CNN
-F 1 "GND" H 20530 8852 50  0000 C CNN
-F 2 "" H 20525 9025 50  0001 C CNN
-F 3 "" H 20525 9025 50  0001 C CNN
-	1    20525 9025
-	1    0    0    -1
-$EndComp
-Wire Wire Line
-	20625 9025 20525 9025
-Wire Wire Line
-	20625 9625 20525 9625
-Wire Wire Line
-	20825 9625 20925 9625
-Wire Wire Line
-	20825 9025 20925 9025
-$Comp
-L Device:R_Small R11
-U 1 1 605942A8
-P 20725 9025
-F 0 "R11" V 20529 9025 50  0000 C CNN
-F 1 "5.1k" V 20620 9025 50  0000 C CNN
-F 2 "Resistor_SMD:R_0805_2012Metric_Pad1.20x1.40mm_HandSolder" H 20725 9025 50  0001 C CNN
-F 3 "~" H 20725 9025 50  0001 C CNN
-	1    20725 9025
-	0    1    1    0
-$EndComp
-$Comp
-L Device:R_Small R12
-U 1 1 605942A2
-P 20725 9625
-F 0 "R12" V 20529 9625 50  0000 C CNN
-F 1 "5.1k" V 20620 9625 50  0000 C CNN
-F 2 "Resistor_SMD:R_0805_2012Metric_Pad1.20x1.40mm_HandSolder" H 20725 9625 50  0001 C CNN
-F 3 "~" H 20725 9625 50  0001 C CNN
-	1    20725 9625
-	0    1    1    0
-$EndComp
-Wire Wire Line
-	20600 9525 20925 9525
-Text GLabel 20600 9525 0    50   Input ~ 0
-D-
-Text GLabel 20600 9325 0    50   Input ~ 0
-D-
-Text GLabel 20925 9425 0    50   Input ~ 0
-D+
-Text GLabel 20925 9225 0    50   Input ~ 0
-D+
-Wire Wire Line
-	20925 9325 20600 9325
-$Comp
-L power:GND #PWR0116
-U 1 1 60594296
-P 20925 9925
-F 0 "#PWR0116" H 20925 9675 50  0001 C CNN
-F 1 "GND" H 20930 9752 50  0000 C CNN
-F 2 "" H 20925 9925 50  0001 C CNN
-F 3 "" H 20925 9925 50  0001 C CNN
-	1    20925 9925
-	1    0    0    -1
-$EndComp
-Wire Wire Line
-	20925 8525 20800 8525
-$Comp
-L power:GND #PWR0115
-U 1 1 6059428C
-P 20800 8525
-F 0 "#PWR0115" H 20800 8275 50  0001 C CNN
-F 1 "GND" H 20805 8352 50  0000 C CNN
-F 2 "" H 20800 8525 50  0001 C CNN
-F 3 "" H 20800 8525 50  0001 C CNN
-	1    20800 8525
-	1    0    0    -1
-$EndComp
-Wire Wire Line
-	20925 8725 20925 8525
-Wire Wire Line
-	20925 8825 20925 8725
-Connection ~ 20925 8725
-$Comp
-L Type-C:HRO-TYPE-C-31-M-12 USB1
-U 1 1 60594286
-P 21025 9375
-F 0 "USB1" H 20547 9277 60  0000 R CNN
-F 1 "HRO-TYPE-C-31-M-12" V 20547 9383 60  0000 R TNN
-F 2 "Type-C:HRO-TYPE-C-31-M-12-HandSoldering" H 21025 9375 60  0001 C CNN
-F 3 "" H 21025 9375 60  0001 C CNN
-	1    21025 9375
-	-1   0    0    1
-$EndComp
 $Comp
 L Type-C:HRO-TYPE-C-31-M-12 USB?
@@
 	1    0    0    -1
 $EndComp
+Wire Wire Line
+	9000 7400 9100 7400
+Connection ~ 9100 7400
+$Comp
+L power:+5V #PWR?
+U 1 1 60A393A3
+P 9100 7300
+F 0 "#PWR?" H 9100 7150 50  0001 C CNN
+F 1 "+5V" H 9115 7473 50  0000 C CNN
+F 2 "" H 9100 7300 50  0001 C CNN
+F 3 "" H 9100 7300 50  0001 C CNN
+	1    9100 7300
+	1    0    0    -1
+$EndComp
+Wire Wire Line
+	9100 7300 9100 7400
 $EndSCHEMATC
