File: Hangulator/Hangulator.kicad_pcb (KiCad board)
At the start: 2 copper layers, 120 parts, among them SW1 SW_Push, SW2 SW_Push, U0 ATmega32U4-AU, U1 ATmega32U4-AU, Y1 Crystal_GND24_Small, Y2 Crystal_GND24_Small

Commit message: workin it
Parts:
- removed C10, C3, C8, C9: .1uF, Capacitor_SMD:C_0805_2012Metric_Pad1.18x1.45mm_HandSolder
- removed C11, C6: 10uF, Capacitor_SMD:C_0805_2012Metric_Pad1.18x1.45mm_HandSolder
- removed C12, C13, C4, C5: 22pF, Capacitor_SMD:C_0805_2012Metric_Pad1.18x1.45mm_HandSolder
- removed C14, C7: 1uF, Capacitor_SMD:C_0805_2012Metric_Pad1.18x1.45mm_HandSolder
- removed D1, D10, D11, D12, D13, D14, D15, D16, D17, D18, D19, D2, D20, D21, D22, D23, D24, D25, D26, D27, D28, D29, D3, D30, D31, D32, D33, D34, D35, D36, D37, D38, D39, D4, D40, D41, D42, D5, D6, D7, D8, D9: D_Small, Diode_SMD:D_0805_2012Metric_Pad1.15x1.40mm_HandSolder
- removed F1, F2: 500mA, Fuse:Fuse_1206_3216Metric_Pad1.42x1.75mm_HandSolder
- removed R10, R5, R6, R9: 10k, Resistor_SMD:R_0805_2012Metric_Pad1.20x1.40mm_HandSolder
- removed R11, R12: 5.1k, Resistor_SMD:R_0805_2012Metric_Pad1.20x1.40mm_HandSolder
- removed R7, R8: 22, Resistor_SMD:R_0805_2012Metric_Pad1.20x1.40mm_HandSolder
- removed SW1, SW2: SW_Push, random-keyboard-parts:SKQG-1155865
- removed U0: ATmega32U4-AU, Package_QFP:TQFP-44_10x10mm_P0.8mm
- removed USB0: HRO-TYPE-C-31-M-12, Type-C:HRO-TYPE-C-31-M-12-HandSoldering
- removed Y1, Y2: Crystal_GND24_Small, Crystal:Crystal_SMD_3225-4Pin_3.2x2.5mm_HandSoldering
- added J1: Conn_01x02_Male, Diode_SMD:D_0805_2012Metric_Pad1.15x1.40mm_HandSolder, F.Cu at (252.2, 164.2)
- added J2: Conn_01x02_Male, Diode_SMD:D_0805_2012Metric_Pad1.15x1.40mm_HandSolder, F.Cu at (252.5, 157.4)
- added J3: Conn_01x05_Male, Connector_PinHeader_1.27mm:PinHeader_1x05_P1.27mm_Horizontal, F.Cu at (239.0, 158.0)
- added MX43: Logout, MX_Alps_Hybrid:MX-1U-NoLED, F.Cu at (263.3, 194.8)
- added MX44: 7, MX_Alps_Hybrid:MX-1U-NoLED, F.Cu at (263.3, 213.8)
- added MX45: 4, MX_Alps_Hybrid:MX-1U-NoLED, F.Cu at (263.3, 232.9)
- added MX46: 1, MX_Alps_Hybrid:MX-1U-NoLED, F.Cu at (263.3, 251.9)
- added MX47: 0, MX_Alps_Hybrid:MX-1U-NoLED, F.Cu at (263.3, 271.0)
- added MX48: /, MX_Alps_Hybrid:MX-1U-NoLED, F.Cu at (282.3, 194.8)
- added MX49: 8, MX_Alps_Hybrid:MX-1U-NoLED, F.Cu at (282.3, 213.8)
- added MX50: 5, MX_Alps_Hybrid:MX-1U-NoLED, F.Cu at (282.3, 232.9)
- added MX51: 2, MX_Alps_Hybrid:MX-1U-NoLED, F.Cu at (282.3, 251.9)
- added MX52: 0, MX_Alps_Hybrid:MX-1U-NoLED, F.Cu at (282.3, 271.0)
- added MX53: *, MX_Alps_Hybrid:MX-1U-NoLED, F.Cu at (301.4, 194.8)
- added MX54: 9, MX_Alps_Hybrid:MX-1U-NoLED, F.Cu at (301.4, 213.8)
- added MX55: 6, MX_Alps_Hybrid:MX-1U-NoLED, F.Cu at (301.4, 232.9)
- added MX56: 3, MX_Alps_Hybrid:MX-1U-NoLED, F.Cu at (301.4, 251.9)
- added MX57: ., MX_Alps_Hybrid:MX-1U-NoLED, F.Cu at (301.4, 271.0)
- added MX58: -, MX_Alps_Hybrid:MX-1U-NoLED, F.Cu at (320.4, 194.8)
- added MX59: +, MX_Alps_Hybrid:MX-1U-NoLED, F.Cu at (320.4, 213.8)
- added MX60: ,, MX_Alps_Hybrid:MX-1U-NoLED, F.Cu at (320.4, 232.9)
- added MX61: =, MX_Alps_Hybrid:MX-1U-NoLED, F.Cu at (320.4, 251.9)
- added MX62: Enter, MX_Alps_Hybrid:MX-1U-NoLED, F.Cu at (320.4, 271.0)
- added U2: STM32F072VBTx, Package_QFP:LQFP-100_14x14mm_P0.5mm, F.Cu at (292.0, 174.0)
- C1, C2: value .1uF -> 10uF; footprint Capacitor_SMD:C_0805_2012Metric_Pad1.18x1.45mm_HandSolder -> Capacitor_SMD:C_0603_1608Metric_Pad1.08x0.95mm_HandSolder
- R1, R2: footprint Resistor_SMD:R_0805_2012Metric_Pad1.20x1.40mm_HandSolder -> Resistor_SMD:R_0603_1608Metric_Pad0.98x0.95mm_HandSolder
- R3, R4: value 22 -> 5.1K; footprint Resistor_SMD:R_0805_2012Metric_Pad1.20x1.40mm_HandSolder -> Resistor_SMD:R_0603_1608Metric_Pad0.98x0.95mm_HandSolder
- U1: value ATmega32U4-AU -> AMS1117-3.3; footprint Package_QFP:TQFP-44_10x10mm_P0.8mm -> Package_TO_SOT_SMD:SOT-223-3_TabPin2
- moved MX42 379.3 mm to (455.2, 198.5), turned to 16.49 degrees
- moved MX41 316.2 mm to (449.8, 180.2), turned to 16.49 degrees
- moved MX38 308.0 mm to (430.2, 181.0), turned to 16.49 degrees
- moved MX40 292.4 mm to (444.4, 161.9), turned to 16.49 degrees
- moved MX39 289.9 mm to (435.6, 199.3), turned to 16.49 degrees
- moved MX37 283.1 mm to (424.8, 162.8), turned to 16.49 degrees
- moved MX32 279.8 mm to (392.5, 197.2), turned to 23.99 degrees
- moved MX36 269.4 mm to (413.8, 198.2), turned to 23.99 degrees
- moved MX25 249.7 mm to (360.4, 273.0), turned to 73.48 degrees
- moved MX35 245.3 mm to (406.0, 180.7), turned to 23.99 degrees
- moved MX29 237.0 mm to (368.7, 255.0), turned to 57.07 degrees
- moved MX34 222.1 mm to (398.3, 163.3), turned to 23.99 degrees
- moved MX28 221.6 mm to (380.9, 218.0), turned to 23.99 degrees
- moved MX31 208.6 mm to (384.7, 179.8), turned to 23.99 degrees
- moved MX21 204.0 mm to (223.6, 273.0), turned to -73.48 degrees
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Connections:
- C2 pad 1: +5V -> +3V3
- MX1 pad 1: C0.0 -> TAB
- MX1 pad 2: Net-(D1-Pad2) -> GND
- MX10 pad 1: C0.3 -> E
- MX10 pad 2: Net-(D10-Pad2) -> GND
- MX11 pad 1: C0.3 -> D
- MX11 pad 2: Net-(D11-Pad2) -> GND
- MX12 pad 1: C0.3 -> C
- MX12 pad 2: Net-(D12-Pad2) -> GND
- MX13 pad 1: C0.3 -> SPACE
- MX13 pad 2: Net-(D13-Pad2) -> GND
- MX14 pad 1: C0.4 -> R
- MX14 pad 2: Net-(D14-Pad2) -> GND
- MX15 pad 1: C0.4 -> F
- MX15 pad 2: Net-(D15-Pad2) -> GND
- MX16 pad 1: C0.4 -> V
- MX16 pad 2: Net-(D16-Pad2) -> GND
- MX17 pad 1: C0.4 -> M3
- MX17 pad 2: Net-(D17-Pad2) -> GND
- MX18 pad 1: C0.5 -> T
- MX18 pad 2: Net-(D18-Pad2) -> GND
- MX19 pad 1: C0.5 -> G
- MX19 pad 2: Net-(D19-Pad2) -> GND
- MX2 pad 1: C0.0 -> LCTRL
- MX2 pad 2: Net-(D2-Pad2) -> GND
- MX20 pad 1: C0.5 -> B
- MX20 pad 2: Net-(D20-Pad2) -> GND
- MX21 pad 1: C0.5 -> GUI
- MX21 pad 2: Net-(D21-Pad2) -> GND
- MX22 pad 1: C1.5 -> Y
- MX22 pad 2: Net-(D22-Pad2) -> GND
- MX23 pad 1: C1.5 -> H
- MX23 pad 2: Net-(D23-Pad2) -> GND
- MX24 pad 1: C1.5 -> N
- MX24 pad 2: Net-(D24-Pad2) -> GND
- MX25 pad 1: C1.5 -> RT3
- MX25 pad 2: Net-(D25-Pad2) -> GND
- MX26 pad 1: C1.4 -> U
- MX26 pad 2: Net-(D26-Pad2) -> GND
- MX27 pad 1: C1.4 -> J
- MX27 pad 2: Net-(D27-Pad2) -> GND
- MX28 pad 1: C1.4 -> M
- MX28 pad 2: Net-(D28-Pad2) -> GND
- MX29 pad 1: C1.4 -> RT2
- MX29 pad 2: Net-(D29-Pad2) -> GND
- MX3 pad 1: C0.0 -> RSHFT
- MX3 pad 2: Net-(D3-Pad2) -> GND
- MX30 pad 1: C1.3 -> I
- MX30 pad 2: Net-(D30-Pad2) -> GND
- MX31 pad 1: C1.3 -> K
- MX31 pad 2: Net-(D31-Pad2) -> GND
- MX32 pad 1: C1.3 -> ,<
- MX32 pad 2: Net-(D32-Pad2) -> GND
- MX33 pad 1: C1.3 -> RT1
- MX33 pad 2: Net-(D33-Pad2) -> GND
- MX34 pad 1: C1.2 -> O
- MX34 pad 2: Net-(D34-Pad2) -> GND
- MX35 pad 1: C1.2 -> L
- MX35 pad 2: Net-(D35-Pad2) -> GND
- MX36 pad 1: C1.2 -> .>
- MX36 pad 2: Net-(D36-Pad2) -> GND
- MX37 pad 1: C1.1 -> P
- MX37 pad 2: Net-(D37-Pad2) -> GND
- MX38 pad 1: C1.1 -> ;:
- MX38 pad 2: Net-(D38-Pad2) -> GND
- MX39 pad 1: C1.1 -> /?
- MX39 pad 2: Net-(D39-Pad2) -> GND
- MX4 pad 1: C0.1 -> Q
- MX4 pad 2: Net-(D4-Pad2) -> GND
- MX40 pad 1: C1.0 -> BKSPC
- MX40 pad 2: Net-(D40-Pad2) -> GND
- MX41 pad 1: C1.0 -> ENTER
- MX41 pad 2: Net-(D41-Pad2) -> GND
- MX42 pad 1: C1.0 -> LSHFT
- MX42 pad 2: Net-(D42-Pad2) -> GND
- MX5 pad 1: C0.1 -> A
- MX5 pad 2: Net-(D5-Pad2) -> GND
- MX6 pad 1: C0.1 -> Z
- MX6 pad 2: Net-(D6-Pad2) -> GND
- MX7 pad 1: C0.2 -> W
- MX7 pad 2: Net-(D7-Pad2) -> GND
- MX8 pad 1: C0.2 -> S
- MX8 pad 2: Net-(D8-Pad2) -> GND
- MX9 pad 1: C0.2 -> X
- MX9 pad 2: Net-(D9-Pad2) -> GND
- R1 pad 1: Net-(R1-Pad1) -> GND
- R2 pad 1: Net-(R2-Pad1) -> GND
- R2 pad 2: Net-(R1-Pad2) -> Net-(R2-Pad2)
- R3 pad 1: Net-(R3-Pad1) -> +3V3
- R3 pad 2: D0+ -> RESET
- R4 pad 1: Net-(R4-Pad1) -> BOOT
- R4 pad 2: D0- -> GND
- U1 pad 1: Net-(U1-Pad1) -> GND
- U1 pad 2: +5V -> +3V3
- U1 pad 3: Net-(R8-Pad1) -> +5V
- USB1 pad 10: Net-(R11-Pad1) -> Net-(R2-Pad2)
- USB1 pad 11: Net-(F2-Pad1) -> +5V
- USB1 pad 2: Net-(F2-Pad1) -> +5V
- USB1 pad 3: Net-(USB1-Pad3) -> unconnected-(USB1-Pad3)
- USB1 pad 4: Net-(R12-Pad1) -> Net-(R1-Pad2)
- USB1 pad 9: Net-(USB1-Pad9) -> unconnected-(USB1-Pad9)
Routing:
- net RSHFT: track 0.00 -> 195.2 mm
- net LSHFT: track 0.00 -> 187.6 mm
- net LCTRL: track 0.00 -> 176.9 mm
- net Z: track 0.00 -> 176.8 mm
- net +3V3: track 0.00 -> 171.1 mm, vias 0 -> 8
- net ENTER: track 0.00 -> 168.0 mm
- net TAB: track 0.00 -> 161.7 mm
- net /?: track 0.00 -> 161.2 mm
- net A: track 0.00 -> 154.7 mm
- net BKSPC: track 0.00 -> 151.7 mm
- net X: track 0.00 -> 149.8 mm
- net ;:: track 0.00 -> 143.9 mm
- net Q: track 0.00 -> 141.9 mm
- net .>: track 0.00 -> 133.5 mm
- net RT3: track 0.00 -> 132.7 mm
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- added copper zone on F.Cu, net GND
Other:
- board outline added: 350 x 136.5 mm
- net class Default removed

Commit message: made some more headway
Parts:
- removed J3: Conn_01x05_Male, Connector_PinHeader_1.27mm:PinHeader_1x05_P1.27mm_Horizontal
- added G***: LOGO, Hangulator-backups:galaxy_silkscreen, F.Cu at (292.1, 215.9)
- added TP1: TestPoint_Small, TestPoint:TestPoint_Pad_D1.0mm, F.Cu at (238.8, 157.9)
- added TP2: TestPoint_Small, TestPoint:TestPoint_Pad_D1.0mm, F.Cu at (233.7, 157.9)
- added TP3: TestPoint_Small, TestPoint:TestPoint_Pad_D1.0mm, F.Cu at (236.3, 157.9)
- added TP4: TestPoint_Small, TestPoint:TestPoint_Pad_D1.0mm, F.Cu at (238.9, 161.3)
- added TP5: TestPoint_Small, TestPoint:TestPoint_Pad_D1.0mm, F.Cu at (233.7, 161.4)
- moved R2 2.24 mm to (283.6, 155.5), turned to 90 degrees
- moved R1 1.78 mm to (299.1, 155.5), turned to 90 degrees
Routing:
- net +5V: track 44.4 -> 63.8 mm, vias 2 -> 3
- net GND: track 80.7 -> 77.6 mm
- net Net-(R2-Pad2): track 7.39 -> 9.72 mm
- net .>: track 133.5 -> 135.1 mm
- net SWCLK: track 64.8 -> 63.9 mm
- net SWDIO: track 70.5 -> 69.8 mm
Other:
- rule pad_to_mask_clearance: 0 -> 0.2

Commit message: mORE lol
Parts:
- added C10: 4.7uF, Capacitor_SMD:C_0603_1608Metric_Pad1.08x0.95mm_HandSolder, B.Cu at (316.6, 157.9)
- added C3: 100nF, Capacitor_SMD:C_0805_2012Metric_Pad1.18x1.45mm_HandSolder, B.Cu at (286.0, 167.2)
- added C4: 100nF, Capacitor_SMD:C_0805_2012Metric_Pad1.18x1.45mm_HandSolder, B.Cu at (298.6, 167.9)
- added C5: 100nF, Capacitor_SMD:C_0805_2012Metric_Pad1.18x1.45mm_HandSolder, B.Cu at (299.1, 178.9)
- added C6: 100nF, Capacitor_SMD:C_0805_2012Metric_Pad1.18x1.45mm_HandSolder, B.Cu at (285.4, 180.0)
- added C7: 10nF, Capacitor_SMD:C_0805_2012Metric_Pad1.18x1.45mm_HandSolder, B.Cu at (296.0, 180.8)
- added C8: 1uF, Capacitor_SMD:C_0805_2012Metric_Pad1.18x1.45mm_HandSolder, B.Cu at (299.9, 181.8)
- added C9: 4.7uF, Capacitor_SMD:C_0603_1608Metric_Pad1.08x0.95mm_HandSolder, B.Cu at (292.4, 163.1)
- C1, C2: footprint Capacitor_SMD:C_0603_1608Metric_Pad1.08x0.95mm_HandSolder -> Capacitor_SMD:C_0805_2012Metric_Pad1.18x1.45mm_HandSolder; moved to B.Cu
- R1, R2, R3, R4: footprint Resistor_SMD:R_0603_1608Metric_Pad0.98x0.95mm_HandSolder -> Resistor_SMD:R_0805_2012Metric_Pad1.20x1.40mm_HandSolder
- U1: moved to B.Cu
- moved C1 13.9 mm to (307.1, 155.7)
- moved C2 13.4 mm to (320.9, 158.1), turned to -90 degrees
- moved U1 1.52 mm to (329.2, 157.0), turned to 0 degrees
Connections:
- U2 pad 100: +3V3 -> VDD1
- U2 pad 21: +3V3 -> VDDA
- U2 pad 28: +3V3 -> VDD1
- U2 pad 40: I -> .>
- U2 pad 41: .> -> I
- U2 pad 50: +3V3 -> VDD1
- U2 pad 6: +3V3 -> VDD1
- U2 pad 75: +3V3 -> VDDIO2
Routing:
- net VDD1: track 0.00 -> 178.2 mm, vias 0 -> 7
- net +3V3: track 171.1 -> 0.00 mm, vias 8 -> 0
- net .>: track 135.1 -> 119.8 mm
- net E: track 106.2 -> 92.2 mm
- net RESET: track 64.4 -> 70.7 mm
- net +5V: track 63.8 -> 61.3 mm, vias 3 -> 2
- net GND: track 77.6 -> 75.2 mm
- net I: track 77.5 -> 78.7 mm
- added copper zone on B.Cu, net GND

Commit message: Done did it now, sent to the man to  make
Parts:
- added ?: , , F.Cu at (347.5, 157.5)
- added ?: , , F.Cu at (242.5, 240.0)
- added ?: , , F.Cu at (397.5, 207.5)
- added ?: , , F.Cu at (267.5, 152.5)
- added ?: , , F.Cu at (340.0, 242.5)
- added REF**: Pin_D1.0mm_L10.0mm_LooseFit, Connector_Pin:Pin_D1.0mm_L10.0mm_LooseFit, F.Cu at (187.5, 207.5)
- moved R1 1.90 mm to (299.1, 153.6), turned to -90 degrees
Connections:
- C2 pad 1: +3V3 -> VDD1
- C6 pad 2: VDDIO2 -> VDD1
- C7 pad 2: VDDA -> VDD1
- C8 pad 2: VDDA -> VDD1
- C9 pad 2: VDDIO2 -> VDD1
- J2 pad 1: +3V3 -> VDD1
- R3 pad 1: +3V3 -> VDD1
- TP1 pad 1: +3V3 -> VDD1
- U1 pad 2: +3V3 -> VDD1
- U2 pad 21: VDDA -> VDD1
- U2 pad 75: VDDIO2 -> VDD1
Routing:
- net /: track 30.8 -> 15.2 mm
- net GND: track 75.2 -> 78.0 mm, vias 2 -> 3
