File: Hangulator/Hangulator.kicad_sch (KiCad schematic)
At the start: 74 parts, among them J1 Conn_01x02_Male, J2 Conn_01x02_Male, J3 Conn_01x05_Male, U1 AMS1117-3.3, U2 STM32F072VBTx

Commit message: made some more headway
Parts:
- removed J3: Conn_01x05_Male, Connector_PinHeader_1.27mm:PinHeader_1x05_P1.27mm_Horizontal, symbol Connector:Conn_01x05_Male
- added TP1, TP2, TP3, TP4, TP5: TestPoint_Small, TestPoint:TestPoint_Pad_D1.0mm, symbol Connector:TestPoint_Small
Connections:
- net +3V3: now also TP1.1
- net 00: now also U2.12 (PF0); no longer U2.11 (PF10)
- net 01: now also U2.5 (PE6); no longer U2.7 (PC13)
- net 1: now also U2.4 (PE5); no longer U2.5 (PE6)
- net 2: now also U2.11 (PF10); no longer U2.10 (PF9)
- net 4: now also U2.3 (PE4); no longer U2.4 (PE5)
- net 5: now also U2.10 (PF9); no longer U2.73 (PF6)
- net 7: now also MX44.1 (COL), U2.2 (PE3); no longer MX49.1 (COL), U2.3 (PE4)
- net 8: now also MX49.1 (COL)
- net GND: now also TP5.1
- net LOGOUT: now also U2.1 (PE2); no longer U2.2 (PE3)
- net PC1: now also U2.13 (PF1); no longer U2.12 (PF0)
- net PC3: no longer U2.78 (PC10), U2.79 (PC11), U2.80 (PC12)
- net RESET: now also TP4.1
- net SWCLK: now also TP2.1
- net SWDIO: now also TP3.1
- net TAB: now reaches MX1.1 (COL)
- net TAB: now also U2.77 (PA15)
- net Q: now reaches MX4.1 (COL)
- net Q: now also U2.80 (PC12)
- net W: now reaches MX7.1 (COL)
- net W: now also U2.83 (PD2)
- net E: now reaches MX10.1 (COL)
- net E: now also U2.86 (PD5)
- net R: now reaches MX14.1 (COL)
- net R: now also U2.89 (PB3)
- net T: now reaches MX18.1 (COL)
- net T: now also U2.92 (PB6)
- net LCTRL: now reaches MX2.1 (COL)
- net LCTRL: now also U2.78 (PC10)
- net A: now reaches MX5.1 (COL)
- net A: now also U2.81 (PD0)
- net S: now reaches MX8.1 (COL)
- net S: now also U2.84 (PD3)
- net D: now reaches MX11.1 (COL)
- net D: now also U2.87 (PD6)
- net F: now reaches MX15.1 (COL)
- net F: now also U2.90 (PB4)
- net G: now reaches MX19.1 (COL)
- net G: now also U2.95 (PB8)
- net RSHFT: now reaches MX3.1 (COL)
- net RSHFT: now also U2.79 (PC11)
- net Z: now reaches MX6.1 (COL)
- net Z: now also U2.82 (PD1)
- net X: now reaches MX9.1 (COL)
- net X: now also U2.85 (PD4)
- net C: now reaches MX12.1 (COL)
- net C: now also U2.88 (PD7)
- net V: now reaches MX16.1 (COL)
- net V: now also U2.91 (PB5)
- net B: now reaches MX20.1 (COL)
- net B: now also U2.96 (PB9)
- net SPACE: now reaches MX13.1 (COL)
- net SPACE: now also U2.97 (PE0)
- net M3: now reaches MX17.1 (COL)
- net M3: now also U2.98 (PE1)
- net GUI: now reaches MX21.1 (COL)
- net GUI: now also U2.7 (PC13)
- no-connect marks 0 -> 2

Commit message: lol
Parts:
- added C10, C9: 4.7uF, Capacitor_SMD:C_0603_1608Metric_Pad1.08x0.95mm_HandSolder, symbol Device:C_Small
- added C3, C4, C5, C6: 100nF, Capacitor_SMD:C_0805_2012Metric_Pad1.18x1.45mm_HandSolder, symbol Device:C_Small
- added C7: 10nF, Capacitor_SMD:C_0805_2012Metric_Pad1.18x1.45mm_HandSolder, symbol Device:C_Small
- added C8: 1uF, Capacitor_SMD:C_0805_2012Metric_Pad1.18x1.45mm_HandSolder, symbol Device:C_Small
- C1, C2: footprint Capacitor_SMD:C_0603_1608Metric_Pad1.08x0.95mm_HandSolder -> Capacitor_SMD:C_0805_2012Metric_Pad1.18x1.45mm_HandSolder
- R1, R2, R3, R4: footprint Resistor_SMD:R_0603_1608Metric_Pad0.98x0.95mm_HandSolder -> Resistor_SMD:R_0805_2012Metric_Pad1.20x1.40mm_HandSolder
Connections:
- net +3V3: no longer U2.100 (VDD), U2.21 (VDDA), U2.28 (VDD), U2.50 (VDD), U2.6 (VBAT), U2.75 (VDDIO2)
- net .>: now also U2.40 (PE9); no longer U2.41 (PE10)
- net GND: now also C10.1, C3.1, C4.1, C5.1, C6.1, C7.1, C8.1, C9.1
- net I: now also U2.41 (PE10); no longer U2.40 (PE9)
- new net VDD1: C10.2, C3.2, C4.2, C5.2, U2.100 (VDD), U2.28 (VDD), U2.50 (VDD), U2.6 (VBAT)
- new net VDDA: C7.2, C8.2, U2.21 (VDDA)
- new net VDDIO2: C6.2, C9.2, U2.75 (VDDIO2)
Other:
- moved on the sheet: U2

Commit message: Done did it now, sent to the man to  make
Connections:
- net VDD1 is gone; now on net +3V3: C10.2, C3.2, C4.2, C5.2, U2.100 (VDD), U2.28 (VDD), U2.50 (VDD), U2.6 (VBAT)
- net VDDA is gone; now on net +3V3: C7.2, C8.2, U2.21 (VDDA)
- net VDDIO2 is gone; now on net +3V3: C6.2, C9.2, U2.75 (VDDIO2)
Changed lines of the file:
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@@
   (junction (at 330.2 58.42) (diameter 1.016) (color 0 0 0 0))
   (junction (at 332.74 41.91) (diameter 1.016) (color 0 0 0 0))
+  (junction (at 334.01 63.5) (diameter 1.016) (color 0 0 0 0))
   (junction (at 334.01 77.47) (diameter 1.016) (color 0 0 0 0))
+  (junction (at 344.17 44.45) (diameter 1.016) (color 0 0 0 0))
+  (junction (at 345.44 78.74) (diameter 1.016) (color 0 0 0 0))
+  (junction (at 346.71 63.5) (diameter 1.016) (color 0 0 0 0))
   (junction (at 346.71 241.3) (diameter 1.016) (color 0 0 0 0))
   (junction (at 349.25 241.3) (diameter 1.016) (color 0 0 0 0))
+  (junction (at 351.79 63.5) (diameter 1.016) (color 0 0 0 0))
   (junction (at 351.79 241.3) (diameter 1.016) (color 0 0 0 0))
   (junction (at 354.33 241.3) (diameter 1.016) (color 0 0 0 0))
@@
     (stroke (width 0) (type solid) (color 0 0 0 0))
   )
-  (wire (pts (xy 334.01 58.42) (xy 334.01 69.85))
+  (wire (pts (xy 334.01 58.42) (xy 334.01 63.5))
+    (stroke (width 0) (type solid) (color 0 0 0 0))
+  )
+  (wire (pts (xy 334.01 63.5) (xy 334.01 69.85))
+    (stroke (width 0) (type solid) (color 0 0 0 0))
+  )
+  (wire (pts (xy 334.01 63.5) (xy 346.71 63.5))
     (stroke (width 0) (type solid) (color 0 0 0 0))
   )
@@
     (stroke (width 0) (type solid) (color 0 0 0 0))
   )
-  (wire (pts (xy 344.17 38.1) (xy 344.17 49.53))
+  (wire (pts (xy 344.17 38.1) (xy 344.17 44.45))
+    (stroke (width 0) (type solid) (color 0 0 0 0))
+  )
+  (wire (pts (xy 344.17 44.45) (xy 344.17 49.53))
     (stroke (width 0) (type solid) (color 0 0 0 0))
   )
@@
     (stroke (width 0) (type solid) (color 0 0 0 0))
   )
-  (wire (pts (xy 345.44 74.93) (xy 345.44 83.82))
+  (wire (pts (xy 345.44 74.93) (xy 345.44 78.74))
+    (stroke (width 0) (type solid) (color 0 0 0 0))
+  )
+  (wire (pts (xy 345.44 78.74) (xy 345.44 83.82))
     (stroke (width 0) (type solid) (color 0 0 0 0))
   )
@@
     (stroke (width 0) (type solid) (color 0 0 0 0))
   )
+  (wire (pts (xy 346.71 62.23) (xy 346.71 63.5))
+    (stroke (width 0) (type solid) (color 0 0 0 0))
+  )
+  (wire (pts (xy 346.71 63.5) (xy 351.79 63.5))
+    (stroke (width 0) (type solid) (color 0 0 0 0))
+  )
   (wire (pts (xy 346.71 101.6) (xy 349.25 101.6))
     (stroke (width 0) (type solid) (color 0 0 0 0))
@@
     (stroke (width 0) (type solid) (color 0 0 0 0))
   )
+  (wire (pts (xy 351.79 44.45) (xy 344.17 44.45))
+    (stroke (width 0) (type solid) (color 0 0 0 0))
+  )
+  (wire (pts (xy 351.79 63.5) (xy 351.79 44.45))
+    (stroke (width 0) (type solid) (color 0 0 0 0))
+  )
+  (wire (pts (xy 351.79 63.5) (xy 351.79 78.74))
+    (stroke (width 0) (type solid) (color 0 0 0 0))
+  )
+  (wire (pts (xy 351.79 78.74) (xy 345.44 78.74))
+    (stroke (width 0) (type solid) (color 0 0 0 0))
+  )
   (wire (pts (xy 351.79 241.3) (xy 349.25 241.3))
     (stroke (width 0) (type solid) (color 0 0 0 0))
@@
     (pin "1")
   )
+  (symbol (lib_id "power:+3V3") (at 346.71 62.23 0) (unit 1)
+    (in_bom yes) (on_board yes)
+    (property "Reference" "#PWR0101" (id 0) (at 346.71 66.04 0)
+      (effects (font (size 1.27 1.27)) hide)
+    )
+    (property "Value" "+3V3" (id 1) (at 347.0783 57.9056 0))
+    (property "Footprint" "" (id 2) (at 346.71 62.23 0)
+      (effects (font (size 1.27 1.27)) hide)
+    )
+    (property "Datasheet" "" (id 3) (at 346.71 62.23 0)
+      (effects (font (size 1.27 1.27)) hide)
+    )
+    (pin "1")
+  )
   (symbol (lib_id "power:GND") (at 40.64 43.18 0) (unit 1)
     (in_bom yes) (on_board yes)
@@
       (reference "#PWR076") (unit 1) (value "GND") (footprint "")
     )
+    (path "/7347d0e4-d6fb-4a3f-95e3-0de11a746784"
+      (reference "#PWR0101") (unit 1) (value "+3V3") (footprint "")
+    )
     (path "/796b03cf-f605-4d38-b566-697d17fd39b0"
